File: _saved_besc g2 mcu.sch (KiCad schematic (older format))
At the start: 37 parts, among them U7 SN74LVC1G04, U8 STM32F405RGTx, Y1 Crystal

Commit message: layout and routing progress
Parts:
- C63: value C_Small -> 100n
Changed lines of the file:
@@
 P 2650 5600
 F 0 "C63" H 2742 5646 50  0000 L CNN
-F 1 "C_Small" H 2742 5555 50  0000 L CNN
+F 1 "100n" H 2742 5555 50  0000 L CNN
 F 2 "Capacitor_SMD:C_0603_1608Metric" H 2650 5600 50  0001 C CNN
 F 3 "~" H 2650 5600 50  0001 C CNN
