File: besc g2 pwr mng.sch (KiCad schematic (older format))
At the start: 11 parts

Commit message: power stage layout draft
Parts:
- C89, C92, C93, C94, C95: renamed from C?; footprint (none) -> Capacitor_SMD:C_0603_1608Metric
- C90, C91: renamed from C?; footprint (none) -> Capacitor_Tantalum_SMD:CP_EIA-6032-28_Kemet-C
- FB8: renamed from FB?; footprint (none) -> Inductor_SMD:L_0603_1608Metric
- J16: renamed from J?; footprint (none) -> Connector_PinHeader_2.54mm:PinHeader_1x02_P2.54mm_Vertical
- gave numbers to parts that had none: 2
Changed lines of the file:
@@
 $EndDescr
 $Comp
-L Regulator_Switching:R-78S3.3-0.1 U?
+L Regulator_Switching:R-78S3.3-0.1 U8
 U 1 1 5DBE4AF8
 P 3200 2450
-F 0 "U?" H 3200 2792 50  0000 C CNN
+F 0 "U8" H 3200 2792 50  0000 C CNN
 F 1 "R-78S3.3-0.1" H 3200 2701 50  0000 C CNN
 F 2 "Converter_DCDC:Converter_DCDC_RECOM_R-78S-0.1_THT" H 3250 2200 50  0001 L CIN
@@
 $EndComp
 $Comp
-L power:+12V #PWR0178
+L power:+12V #PWR0123
 U 1 1 5DBE7656
 P 1750 2300
-F 0 "#PWR0178" H 1750 2150 50  0001 C CNN
+F 0 "#PWR0123" H 1750 2150 50  0001 C CNN
 F 1 "+12V" H 1765 2473 50  0000 C CNN
 F 2 "" H 1750 2300 50  0001 C CNN
@@
 	2800 2350 2550 2350
 $Comp
-L Device:Ferrite_Bead_Small FB?
+L Device:Ferrite_Bead_Small FB8
 U 1 1 5DBE82BD
 P 1950 2350
-F 0 "FB?" V 1713 2350 50  0000 C CNN
+F 0 "FB8" V 1713 2350 50  0000 C CNN
 F 1 "fb" V 1804 2350 50  0000 C CNN
-F 2 "" V 1880 2350 50  0001 C CNN
+F 2 "Inductor_SMD:L_0603_1608Metric" V 1880 2350 50  0001 C CNN
 F 3 "~" H 1950 2350 50  0001 C CNN
 	1    1950 2350
@@
 $EndComp
 $Comp
-L Device:C_Small C?
+L Device:C_Small C92
 U 1 1 5DBE8B52
 P 2550 2500
-F 0 "C?" H 2642 2546 50  0000 L CNN
+F 0 "C92" H 2642 2546 50  0000 L CNN
 F 1 "2.2u" H 2642 2455 50  0000 L CNN
-F 2 "" H 2550 2500 50  0001 C CNN
+F 2 "Capacitor_SMD:C_0603_1608Metric" H 2550 2500 50  0001 C CNN
 F 3 "~" H 2550 2500 50  0001 C CNN
 	1    2550 2500
@@
 	2150 2400 2150 2350
 $Comp
-L power:GNDD #PWR0179
+L power:GNDD #PWR0128
 U 1 1 5DBE9845
 P 2550 2650
-F 0 "#PWR0179" H 2550 2400 50  0001 C CNN
+F 0 "#PWR0128" H 2550 2400 50  0001 C CNN
 F 1 "GNDD" H 2554 2495 50  0000 C CNN
 F 2 "" H 2550 2650 50  0001 C CNN
@@
 $EndComp
 $Comp
-L power:GNDD #PWR0180
+L power:GNDD #PWR0129
 U 1 1 5DBE9BC8
 P 3200 2800
-F 0 "#PWR0180" H 3200 2550 50  0001 C CNN
+F 0 "#PWR0129" H 3200 2550 50  0001 C CNN
 F 1 "GNDD" H 3204 2645 50  0000 C CNN
 F 2 "" H 3200 2800 50  0001 C CNN
@@
 	2550 2600 2550 2650
 $Comp
-L Device:C_Small C?
+L Device:C_Small C89
 U 1 1 5DBEA31C
 P 1750 2500
-F 0 "C?" H 1842 2546 50  0000 L CNN
+F 0 "C89" H 1842 2546 50  0000 L CNN
 F 1 "2.2u" H 1842 2455 50  0000 L CNN
-F 2 "" H 1750 2500 50  0001 C CNN
+F 2 "Capacitor_SMD:C_0603_1608Metric" H 1750 2500 50  0001 C CNN
 F 3 "~" H 1750 2500 50  0001 C CNN
 	1    1750 2500
@@
 	1750 2350 1750 2400
 $Comp
-L power:GND #PWR0181
+L power:GND #PWR0124
 U 1 1 5DBEAD9C
 P 1750 2650
-F 0 "#PWR0181" H 1750 2400 50  0001 C CNN
+F 0 "#PWR0124" H 1750 2400 50  0001 C CNN
 F 1 "GND" H 1755 2477 50  0000 C CNN
 F 2 "" H 1750 2650 50  0001 C CNN
@@
 	2550 2400 2550 2350
 $Comp
-L Device:CP_Small C?
+L Device:CP_Small C90
 U 1 1 5DBEE8A0
 P 2150 2500
-F 0 "C?" H 2238 2546 50  0000 L CNN
+F 0 "C90" H 2238 2546 50  0000 L CNN
 F 1 "100u" H 2238 2455 50  0000 L CNN
-F 2 "" H 2150 2500 50  0001 C CNN
+F 2 "Capacitor_Tantalum_SMD:CP_EIA-6032-28_Kemet-C" H 2150 2500 50  0001 C CNN
 F 3 "~" H 2150 2500 50  0001 C CNN
 F 4 "TAJD107M016RNJ" H 2150 2500 50  0001 C CNN "PART"
@@
 $EndComp
 $Comp
-L power:GNDD #PWR0182
+L power:GNDD #PWR0125
 U 1 1 5DBEEAFF
 P 2150 2650
-F 0 "#PWR0182" H 2150 2400 50  0001 C CNN
+F 0 "#PWR0125" H 2150 2400 50  0001 C CNN
 F 1 "GNDD" H 2154 2495 50  0000 C CNN
 F 2 "" H 2150 2650 50  0001 C CNN
@@
 Connection ~ 2550 2350
 $Comp
-L power:+5V #PWR0183
+L power:+5V #PWR0130
 U 1 1 5DBEF49F
 P 3650 2400
-F 0 "#PWR0183" H 3650 2250 50  0001 C CNN
+F 0 "#PWR0130" H 3650 2250 50  0001 C CNN
 F 1 "+5V" H 3665 2573 50  0000 C CNN
 F 2 "" H 3650 2400 50  0001 C CNN
@@
 	3650 2450 3650 2400
 $Comp
-L Regulator_Linear:LP5907MFX-3.3 U?
+L Regulator_Linear:LP5907MFX-3.3 U9
 U 1 1 5DBF5F54
 P 4900 2500
-F 0 "U?" H 4900 2867 50  0000 C CNN
+F 0 "U9" H 4900 2867 50  0000 C CNN
 F 1 "LP5907MFX-3.3" H 4900 2776 50  0000 C CNN
 F 2 "Package_TO_SOT_SMD:SOT-23-5" H 4900 2850 50  0001 C CNN
@@
 $EndComp
 $Comp
-L Device:C_Small C?
+L Device:C_Small C93
 U 1 1 5DBF66B9
 P 4250 2550
-F 0 "C?" H 4342 2596 50  0000 L CNN
+F 0 "C93" H 4342 2596 50  0000 L CNN
 F 1 "2.2u" H 4342 2505 50  0000 L CNN
-F 2 "" H 4250 2550 50  0001 C CNN
+F 2 "Capacitor_SMD:C_0603_1608Metric" H 4250 2550 50  0001 C CNN
 F 3 "~" H 4250 2550 50  0001 C CNN
 	1    4250 2550
@@
 $EndComp
 $Comp
-L Device:C_Small C?
+L Device:C_Small C94
 U 1 1 5DBF6D06
 P 5400 2550
-F 0 "C?" H 5492 2596 50  0000 L CNN
+F 0 "C94" H 5492 2596 50  0000 L CNN
 F 1 "2.2u" H 5492 2505 50  0000 L CNN
-F 2 "" H 5400 2550 50  0001 C CNN
+F 2 "Capacitor_SMD:C_0603_1608Metric" H 5400 2550 50  0001 C CNN
 F 3 "~" H 5400 2550 50  0001 C CNN
 	1    5400 2550
@@
 $EndComp
 $Comp
-L Device:C_Small C?
+L Device:C_Small C95
 U 1 1 5DBF704C
 P 5750 2550
-F 0 "C?" H 5842 2596 50  0000 L CNN
+F 0 "C95" H 5842 2596 50  0000 L CNN
 F 1 "2.2u" H 5842 2505 50  0000 L CNN
-F 2 "" H 5750 2550 50  0001 C CNN
+F 2 "Capacitor_SMD:C_0603_1608Metric" H 5750 2550 50  0001 C CNN
 F 3 "~" H 5750 2550 50  0001 C CNN
 	1    5750 2550
@@
 $EndComp
 $Comp
-L power:GNDD #PWR0184
+L power:GNDD #PWR0133
 U 1 1 5DBF730C
 P 4900 2850
-F 0 "#PWR0184" H 4900 2600 50  0001 C CNN
+F 0 "#PWR0133" H 4900 2600 50  0001 C CNN
 F 1 "GNDD" H 4904 2695 50  0000 C CNN
 F 2 "" H 4900 2850 50  0001 C CNN
@@
 	4250 2400 4250 2450
 $Comp
-L power:GNDD #PWR0185
+L power:GNDD #PWR0132
 U 1 1 5DBF8640
 P 4250 2700
-F 0 "#PWR0185" H 4250 2450 50  0001 C CNN
+F 0 "#PWR0132" H 4250 2450 50  0001 C CNN
 F 1 "GNDD" H 4254 2545 50  0000 C CNN
 F 2 "" H 4250 2700 50  0001 C CNN
@@
 	5400 2400 5750 2400
 $Comp
-L power:GNDD #PWR0186
+L power:GNDD #PWR0134
 U 1 1 5DBF9740
 P 5400 2750
-F 0 "#PWR0186" H 5400 2500 50  0001 C CNN
+F 0 "#PWR0134" H 5400 2500 50  0001 C CNN
 F 1 "GNDD" H 5404 2595 50  0000 C CNN
 F 2 "" H 5400 2750 50  0001 C CNN
@@
 	5400 2700 5400 2750
 $Comp
-L power:+5V #PWR0187
+L power:+5V #PWR0131
 U 1 1 5DBFA2FB
 P 4250 2350
-F 0 "#PWR0187" H 4250 2200 50  0001 C CNN
+F 0 "#PWR0131" H 4250 2200 50  0001 C CNN
 F 1 "+5V" H 4265 2523 50  0000 C CNN
 F 2 "" H 4250 2350 50  0001 C CNN
@@
 	4250 2350 4250 2400
 $Comp
-L power:+3.3V #PWR0188
+L power:+3.3V #PWR0135
 U 1 1 5DBFAF4E
 P 5750 2350
-F 0 "#PWR0188" H 5750 2200 50  0001 C CNN
+F 0 "#PWR0135" H 5750 2200 50  0001 C CNN
 F 1 "+3.3V" H 5765 2523 50  0000 C CNN
 F 2 "" H 5750 2350 50  0001 C CNN
@@
 Connection ~ 5750 2400
 $Comp
-L Connector_Generic:Conn_01x02 J?
+L Connector_Generic:Conn_01x02 J16
 U 1 1 5DC09E1F
 P 1700 3750
-F 0 "J?" H 1618 3967 50  0000 C CNN
+F 0 "J16" H 1618 3967 50  0000 C CNN
 F 1 "12V IN" H 1618 3876 50  0000 C CNN
-F 2 "" H 1700 3750 50  0001 C CNN
+F 2 "Connector_PinHeader_2.54mm:PinHeader_1x02_P2.54mm_Vertical" H 1700 3750 50  0001 C CNN
 F 3 "~" H 1700 3750 50  0001 C CNN
 	1    1700 3750
@@
 	1900 3850 1900 4050
 $Comp
-L power:GND #PWR0189
+L power:GND #PWR0127
 U 1 1 5DC0C402
 P 2150 4100
-F 0 "#PWR0189" H 2150 3850 50  0001 C CNN
+F 0 "#PWR0127" H 2150 3850 50  0001 C CNN
 F 1 "GND" H 2155 3927 50  0000 C CNN
 F 2 "" H 2150 4100 50  0001 C CNN
@@
 Connection ~ 2150 4050
 $Comp
-L Device:CP_Small C?
+L Device:CP_Small C91
 U 1 1 5DC0CFC2
 P 2150 3900
-F 0 "C?" H 2238 3946 50  0000 L CNN
+F 0 "C91" H 2238 3946 50  0000 L CNN
 F 1 "100u" H 2238 3855 50  0000 L CNN
-F 2 "" H 2150 3900 50  0001 C CNN
+F 2 "Capacitor_Tantalum_SMD:CP_EIA-6032-28_Kemet-C" H 2150 3900 50  0001 C CNN
 F 3 "~" H 2150 3900 50  0001 C CNN
 F 4 "TAJD107M016RNJ" H 2150 3900 50  0001 C CNN "PART"
@@
 $EndComp
 $Comp
-L power:+12V #PWR0190
+L power:+12V #PWR0126
 U 1 1 5DC0D64E
 P 2150 3700
-F 0 "#PWR0190" H 2150 3550 50  0001 C CNN
+F 0 "#PWR0126" H 2150 3550 50  0001 C CNN
 F 1 "+12V" H 2165 3873 50  0000 C CNN
 F 2 "" H 2150 3700 50  0001 C CNN

Commit message: isolated drivers, layout
Parts:
- renumbered C89 to C92, C90 to C93, C91 to C94, C92 to C95, C93 to C96, C94 to C97, C95 to C98, U8 to U11, U9 to U12
Changed lines of the file:
@@
 $EndDescr
 $Comp
-L Regulator_Switching:R-78S3.3-0.1 U8
+L Regulator_Switching:R-78S3.3-0.1 U11
 U 1 1 5DBE4AF8
 P 3200 2450
-F 0 "U8" H 3200 2792 50  0000 C CNN
+F 0 "U11" H 3200 2792 50  0000 C CNN
 F 1 "R-78S3.3-0.1" H 3200 2701 50  0000 C CNN
 F 2 "Converter_DCDC:Converter_DCDC_RECOM_R-78S-0.1_THT" H 3250 2200 50  0001 L CIN
@@
 $EndComp
 $Comp
-L power:+12V #PWR0123
+L power:+12V #PWR0128
 U 1 1 5DBE7656
 P 1750 2300
-F 0 "#PWR0123" H 1750 2150 50  0001 C CNN
+F 0 "#PWR0128" H 1750 2150 50  0001 C CNN
 F 1 "+12V" H 1765 2473 50  0000 C CNN
 F 2 "" H 1750 2300 50  0001 C CNN
@@
 $EndComp
 $Comp
-L Device:C_Small C92
+L Device:C_Small C95
 U 1 1 5DBE8B52
 P 2550 2500
-F 0 "C92" H 2642 2546 50  0000 L CNN
+F 0 "C95" H 2642 2546 50  0000 L CNN
 F 1 "2.2u" H 2642 2455 50  0000 L CNN
 F 2 "Capacitor_SMD:C_0603_1608Metric" H 2550 2500 50  0001 C CNN
@@
 	2150 2400 2150 2350
 $Comp
-L power:GNDD #PWR0128
+L power:GNDD #PWR0133
 U 1 1 5DBE9845
 P 2550 2650
-F 0 "#PWR0128" H 2550 2400 50  0001 C CNN
+F 0 "#PWR0133" H 2550 2400 50  0001 C CNN
 F 1 "GNDD" H 2554 2495 50  0000 C CNN
 F 2 "" H 2550 2650 50  0001 C CNN
@@
 $EndComp
 $Comp
-L power:GNDD #PWR0129
+L power:GNDD #PWR0134
 U 1 1 5DBE9BC8
 P 3200 2800
-F 0 "#PWR0129" H 3200 2550 50  0001 C CNN
+F 0 "#PWR0134" H 3200 2550 50  0001 C CNN
 F 1 "GNDD" H 3204 2645 50  0000 C CNN
 F 2 "" H 3200 2800 50  0001 C CNN
@@
 	2550 2600 2550 2650
 $Comp
-L Device:C_Small C89
+L Device:C_Small C92
 U 1 1 5DBEA31C
 P 1750 2500
-F 0 "C89" H 1842 2546 50  0000 L CNN
+F 0 "C92" H 1842 2546 50  0000 L CNN
 F 1 "2.2u" H 1842 2455 50  0000 L CNN
 F 2 "Capacitor_SMD:C_0603_1608Metric" H 1750 2500 50  0001 C CNN
@@
 	1750 2350 1750 2400
 $Comp
-L power:GND #PWR0124
+L power:GND #PWR0129
 U 1 1 5DBEAD9C
 P 1750 2650
-F 0 "#PWR0124" H 1750 2400 50  0001 C CNN
+F 0 "#PWR0129" H 1750 2400 50  0001 C CNN
 F 1 "GND" H 1755 2477 50  0000 C CNN
 F 2 "" H 1750 2650 50  0001 C CNN
@@
 	2550 2400 2550 2350
 $Comp
-L Device:CP_Small C90
+L Device:CP_Small C93
 U 1 1 5DBEE8A0
 P 2150 2500
-F 0 "C90" H 2238 2546 50  0000 L CNN
+F 0 "C93" H 2238 2546 50  0000 L CNN
 F 1 "100u" H 2238 2455 50  0000 L CNN
 F 2 "Capacitor_Tantalum_SMD:CP_EIA-6032-28_Kemet-C" H 2150 2500 50  0001 C CNN
@@
 $EndComp
 $Comp
-L power:GNDD #PWR0125
+L power:GNDD #PWR0130
 U 1 1 5DBEEAFF
 P 2150 2650
-F 0 "#PWR0125" H 2150 2400 50  0001 C CNN
+F 0 "#PWR0130" H 2150 2400 50  0001 C CNN
 F 1 "GNDD" H 2154 2495 50  0000 C CNN
 F 2 "" H 2150 2650 50  0001 C CNN
@@
 Connection ~ 2550 2350
 $Comp
-L power:+5V #PWR0130
+L power:+5V #PWR0135
 U 1 1 5DBEF49F
 P 3650 2400
-F 0 "#PWR0130" H 3650 2250 50  0001 C CNN
+F 0 "#PWR0135" H 3650 2250 50  0001 C CNN
 F 1 "+5V" H 3665 2573 50  0000 C CNN
 F 2 "" H 3650 2400 50  0001 C CNN
@@
 	3650 2450 3650 2400
 $Comp
-L Regulator_Linear:LP5907MFX-3.3 U9
+L Regulator_Linear:LP5907MFX-3.3 U12
 U 1 1 5DBF5F54
 P 4900 2500
-F 0 "U9" H 4900 2867 50  0000 C CNN
+F 0 "U12" H 4900 2867 50  0000 C CNN
 F 1 "LP5907MFX-3.3" H 4900 2776 50  0000 C CNN
 F 2 "Package_TO_SOT_SMD:SOT-23-5" H 4900 2850 50  0001 C CNN
@@
 $EndComp
 $Comp
-L Device:C_Small C93
+L Device:C_Small C96
 U 1 1 5DBF66B9
 P 4250 2550
-F 0 "C93" H 4342 2596 50  0000 L CNN
+F 0 "C96" H 4342 2596 50  0000 L CNN
 F 1 "2.2u" H 4342 2505 50  0000 L CNN
 F 2 "Capacitor_SMD:C_0603_1608Metric" H 4250 2550 50  0001 C CNN
@@
 $EndComp
 $Comp
-L Device:C_Small C94
+L Device:C_Small C97
 U 1 1 5DBF6D06
 P 5400 2550
-F 0 "C94" H 5492 2596 50  0000 L CNN
+F 0 "C97" H 5492 2596 50  0000 L CNN
 F 1 "2.2u" H 5492 2505 50  0000 L CNN
 F 2 "Capacitor_SMD:C_0603_1608Metric" H 5400 2550 50  0001 C CNN
@@
 $EndComp
 $Comp
-L Device:C_Small C95
+L Device:C_Small C98
 U 1 1 5DBF704C
 P 5750 2550
-F 0 "C95" H 5842 2596 50  0000 L CNN
+F 0 "C98" H 5842 2596 50  0000 L CNN
 F 1 "2.2u" H 5842 2505 50  0000 L CNN
 F 2 "Capacitor_SMD:C_0603_1608Metric" H 5750 2550 50  0001 C CNN
@@
 $EndComp
 $Comp
-L power:GNDD #PWR0133
+L power:GNDD #PWR0138
 U 1 1 5DBF730C
 P 4900 2850
-F 0 "#PWR0133" H 4900 2600 50  0001 C CNN
+F 0 "#PWR0138" H 4900 2600 50  0001 C CNN
 F 1 "GNDD" H 4904 2695 50  0000 C CNN
 F 2 "" H 4900 2850 50  0001 C CNN
@@
 	4250 2400 4250 2450
 $Comp
-L power:GNDD #PWR0132
+L power:GNDD #PWR0137
 U 1 1 5DBF8640
 P 4250 2700
-F 0 "#PWR0132" H 4250 2450 50  0001 C CNN
+F 0 "#PWR0137" H 4250 2450 50  0001 C CNN
 F 1 "GNDD" H 4254 2545 50  0000 C CNN
 F 2 "" H 4250 2700 50  0001 C CNN
@@
 	5400 2400 5750 2400
 $Comp
-L power:GNDD #PWR0134
+L power:GNDD #PWR0139
 U 1 1 5DBF9740
 P 5400 2750
-F 0 "#PWR0134" H 5400 2500 50  0001 C CNN
+F 0 "#PWR0139" H 5400 2500 50  0001 C CNN
 F 1 "GNDD" H 5404 2595 50  0000 C CNN
 F 2 "" H 5400 2750 50  0001 C CNN
@@
 	5400 2700 5400 2750
 $Comp
-L power:+5V #PWR0131
+L power:+5V #PWR0136
 U 1 1 5DBFA2FB
 P 4250 2350
-F 0 "#PWR0131" H 4250 2200 50  0001 C CNN
+F 0 "#PWR0136" H 4250 2200 50  0001 C CNN
 F 1 "+5V" H 4265 2523 50  0000 C CNN
 F 2 "" H 4250 2350 50  0001 C CNN
@@
 	4250 2350 4250 2400
 $Comp
-L power:+3.3V #PWR0135
+L power:+3.3V #PWR0140
 U 1 1 5DBFAF4E
 P 5750 2350
-F 0 "#PWR0135" H 5750 2200 50  0001 C CNN
+F 0 "#PWR0140" H 5750 2200 50  0001 C CNN
 F 1 "+3.3V" H 5765 2523 50  0000 C CNN
 F 2 "" H 5750 2350 50  0001 C CNN
@@
 	1900 3850 1900 4050
 $Comp
-L power:GND #PWR0127
+L power:GND #PWR0132
 U 1 1 5DC0C402
 P 2150 4100
-F 0 "#PWR0127" H 2150 3850 50  0001 C CNN
+F 0 "#PWR0132" H 2150 3850 50  0001 C CNN
 F 1 "GND" H 2155 3927 50  0000 C CNN
 F 2 "" H 2150 4100 50  0001 C CNN
@@
 Connection ~ 2150 4050
 $Comp
-L Device:CP_Small C91
+L Device:CP_Small C94
 U 1 1 5DC0CFC2
 P 2150 3900
-F 0 "C91" H 2238 3946 50  0000 L CNN
+F 0 "C94" H 2238 3946 50  0000 L CNN
 F 1 "100u" H 2238 3855 50  0000 L CNN
 F 2 "Capacitor_Tantalum_SMD:CP_EIA-6032-28_Kemet-C" H 2150 3900 50  0001 C CNN
@@
 $EndComp
 $Comp
-L power:+12V #PWR0126
+L power:+12V #PWR0131
 U 1 1 5DC0D64E
 P 2150 3700
-F 0 "#PWR0126" H 2150 3550 50  0001 C CNN
+F 0 "#PWR0131" H 2150 3550 50  0001 C CNN
 F 1 "+12V" H 2165 3873 50  0000 C CNN
 F 2 "" H 2150 3700 50  0001 C CNN

Commit message: 12V PS, isolated gate drivers
Parts:
- added C100, C101, C102: 0.47u 200V, Capacitor_SMD:C_0603_1608Metric, symbol Device:C_Small
- added C103: 100n, Capacitor_SMD:C_0603_1608Metric, symbol Device:C_Small
- added C104, C105, C106, C107, C108: 4.7u, Capacitor_SMD:C_0603_1608Metric, symbol Device:C_Small
- added C109, C110, C111: 150u, symbol Device:CP_Small
- added C112: 1n, Capacitor_SMD:C_0603_1608Metric, symbol Device:C_Small
- added C113: 10p, Capacitor_SMD:C_0603_1608Metric, symbol Device:C_Small
- added C114: 0.1u, Capacitor_SMD:C_0603_1608Metric, symbol Device:C_Small
- added C115: 2.2u, Capacitor_SMD:C_0603_1608Metric, symbol Device:C_Small
- added C116: 100p, Capacitor_SMD:C_0603_1608Metric, symbol Device:C_Small
- added C117: 4.7n, Capacitor_SMD:C_0603_1608Metric, symbol Device:C_Small
- added C99: 100u, symbol Device:CP_Small
- added D7: D_Zener, symbol Device:D_Zener
- added IC1: LTC7801, Package_DFN_QFN:QFN-24-1EP_4x5mm_P0.5mm_EP2.65x3.65mm, symbol moje:LTC7801
- added L1: INDUCTOR, symbol pspice:INDUCTOR
- added Q25, Q26: Q_NMOS_DGS, symbol Device:Q_NMOS_DGS
- added R80: 8m, Resistor_SMD:R_0603_1608Metric, symbol Device:R_Small
- added R81: 100k, Resistor_SMD:R_0603_1608Metric, symbol Device:R_Small
- added R82: 511k, Resistor_SMD:R_0603_1608Metric, symbol Device:R_Small
- added R83: 10p, Resistor_SMD:R_0603_1608Metric, symbol Device:R_Small
- added R84: 10k, Resistor_SMD:R_0603_1608Metric, symbol Device:R_Small
- added R85: 80k6, Resistor_SMD:R_0603_1608Metric, symbol Device:R_Small
- added R86: 30k1, Resistor_SMD:R_0603_1608Metric, symbol Device:R_Small
- J16: value 12V IN -> 12V OUT
- renumbered C95 to C94, C94 to C95
Connections:
- net labels added: PG, RUN, SENSE+, SENSE-, VDC
- wire segments 41 -> 169
Other:
- moved on the sheet: C92, C93, C94, C95, C96, C97, C98, FB8, J16, U12

Commit message: layout and routing progress
Parts:
- removed C100: 0.47u 200V, Capacitor_SMD:C_0603_1608Metric, symbol Device:C_Small
- removed C103: 100n, Capacitor_SMD:C_0603_1608Metric, symbol Device:C_Small
- removed C106: 4.7u, Capacitor_SMD:C_0603_1608Metric, symbol Device:C_Small
- removed C109, C110, C111: 150u, symbol Device:CP_Small
- removed C113: 10p, Capacitor_SMD:C_0603_1608Metric, symbol Device:C_Small
- removed C115: 2.2u, Capacitor_SMD:C_0603_1608Metric, symbol Device:C_Small
- removed C116: 100p, Capacitor_SMD:C_0603_1608Metric, symbol Device:C_Small
- removed C117: 4.7n, Capacitor_SMD:C_0603_1608Metric, symbol Device:C_Small
- removed C95: 100u, Capacitor_Tantalum_SMD:CP_EIA-6032-28_Kemet-C, symbol Device:CP_Small
- removed C99: 100u, symbol Device:CP_Small
- removed D7: D_Zener, symbol Device:D_Zener
- removed Q25, Q26: Q_NMOS_DGS, symbol Device:Q_NMOS_DGS
- removed R80: 8m, Resistor_SMD:R_0603_1608Metric, symbol Device:R_Small
- removed R81: 100k, Resistor_SMD:R_0603_1608Metric, symbol Device:R_Small
- removed R82: 511k, Resistor_SMD:R_0603_1608Metric, symbol Device:R_Small
- removed R83: 10p, Resistor_SMD:R_0603_1608Metric, symbol Device:R_Small
- removed R84: 10k, Resistor_SMD:R_0603_1608Metric, symbol Device:R_Small
- removed R85: 80k6, Resistor_SMD:R_0603_1608Metric, symbol Device:R_Small
- removed R86: 30k1, Resistor_SMD:R_0603_1608Metric, symbol Device:R_Small
- removed U11: R-78S3.3-0.1, Converter_DCDC:Converter_DCDC_RECOM_R-78S-0.1_THT, symbol Regulator_Switching:R-78S3.3-0.1
- added C110, C111: 4.7u 25V, Capacitor_SMD:C_1206_3216Metric, symbol Device:C_Small
- added C115, C116, C117: TR3D157K016C0075, Capacitor_Tantalum_SMD:CP_EIA-7343-31_Kemet-D, symbol Device:CP_Small
- added C93, C94, C98: 0.47u 200V, Capacitor_SMD:C_1206_3216Metric, symbol Device:C_Small
- added C96: 100n, Capacitor_SMD:C_0603_1608Metric, symbol Device:C_Small
- added C99: 4.7u, Capacitor_SMD:C_0603_1608Metric, symbol Device:C_Small
- added D8: LED, LED_SMD:LED_0603_1608Metric, symbol Device:LED
- added D9: 12.7, Diode_SMD:D_SMA, symbol Device:D_Zener
- added Q25: FDMS86252L, moje:TDSON-8-MOS, symbol Device:Q_NMOS_SGD
- added Q26: BSC110N15NS5, moje:TDSON-8-MOS, symbol Device:Q_NMOS_SGD
- added R87: 470, Resistor_SMD:R_0603_1608Metric, symbol Device:R_Small
- added R88: 1M, Resistor_SMD:R_0603_1608Metric, symbol Device:R_Small
- added R89: 9k1, Resistor_SMD:R_0603_1608Metric, symbol Device:R_Small
- added R90: 100k, Resistor_SMD:R_0603_1608Metric, symbol Device:R_Small
- added R91, R96: 80k6, Resistor_SMD:R_0603_1608Metric, symbol Device:R_Small
- added R92: 10k, Resistor_SMD:R_0603_1608Metric, symbol Device:R_Small
- added R93: 10R, Resistor_SMD:R_0603_1608Metric, symbol Device:R_Small
- added R94: 30k1, Resistor_SMD:R_0603_1608Metric, symbol Device:R_Small
- added R95: 71.5k, Resistor_SMD:R_0603_1608Metric, symbol Device:R_Small
- added R97: 255k, Resistor_SMD:R_0603_1608Metric, symbol Device:R_Small
- added R98: 60k4, Resistor_SMD:R_0603_1608Metric, symbol Device:R_Small
- added R99: 4k32, Resistor_SMD:R_0603_1608Metric, symbol Device:R_Small
- added U11: R-78E5.0-0.5, Converter_DCDC:Converter_DCDC_RECOM_R-78E-0.5_THT, symbol Regulator_Switching:R-78E5.0-0.5
- C100: renamed from C94; value 2.2u -> 4.7u; footprint Capacitor_SMD:C_0603_1608Metric -> Capacitor_SMD:C_1206_3216Metric
- C101: value 0.47u 200V -> 100n 50V
- C102: value 0.47u 200V -> 2.2u 10V
- C104: value 4.7u -> 270p
- C105: value 4.7u -> 130p
- C107: value 4.7u -> 47n
- C108: value 4.7u -> 10p
- C112: value 1n -> 4.7u 25V; footprint Capacitor_SMD:C_0603_1608Metric -> Capacitor_SMD:C_1206_3216Metric
- C114: value 0.1u -> 4.7u 25V; footprint Capacitor_SMD:C_0603_1608Metric -> Capacitor_SMD:C_1206_3216Metric
- C92: value 2.2u -> 0.47u 200V; footprint Capacitor_SMD:C_0603_1608Metric -> Capacitor_SMD:C_1206_3216Metric
- J17: renamed from J16; footprint Connector_PinHeader_2.54mm:PinHeader_1x02_P2.54mm_Vertical -> conn-amass:AMASS_XT30U-M_1x02_P5.0mm_Vertical
- L1: value INDUCTOR -> 7443633300; footprint (none) -> moje:WE-HCF-2013
- renumbered C96 to C103, C97 to C106, C98 to C109, C93 to C97
Connections:
- net labels added: BOTTOM_GATE, DRVSET, FREQ, INTVCC, ITH, OVLO, SS, SW, TOP_GATE, VFB, VIN+
- wire segments 169 -> 179
Other:
- note added: "Freq: 150 kHz"
- note added: "Overvoltage\n133V"
- note added: "possible alternative\nBSC160N15NS5ATMA1"
- note added: "possible alternative\nBSC520N15NS3"
