File: besc g2.kicad_pcb (KiCad board)
At the start: 2 copper layers, 230 x 45 mm, 258 parts, among them J1 Phase, J10 USB_B_Micro, J11 THROTTLE, J12 MOTOR SENSOR, J13 THROTTLE 2 (BRAKE), J14 SERIAL, J15 Conn_01x04, J16 12V IN, J2 Phase, J3 Phase, J4 BUSBAR, J5 BUSBAR, J6 IN+, J7 IN-, J8 SWD, J9 RC PWM, Q1 Q_NMOS_DGS, Q10 Q_NMOS_DGS, Q11 Q_NMOS_DGS, Q12 Q_NMOS_DGS, Q13 Q_NMOS_DGS, Q14 Q_NMOS_DGS, Q15 Q_NMOS_DGS, Q16 Q_NMOS_DGS, Q17 Q_NMOS_DGS, Q18 Q_NMOS_DGS, Q19 Q_NMOS_DGS, Q2 Q_NMOS_DGS, Q20 Q_NMOS_DGS, Q21 Q_NMOS_DGS, Q22 Q_NMOS_DGS, Q23 Q_NMOS_DGS, Q24 Q_NMOS_DGS, Q3 Q_NMOS_DGS, Q4 Q_NMOS_DGS, Q5 Q_NMOS_DGS, Q6 Q_NMOS_DGS, Q7 Q_NMOS_DGS, Q8 Q_NMOS_DGS, Q9 Q_NMOS_DGS, U1 INA240A1D, U2 INA240A1D, U3 INA240A1D, U4 SN74LVC1G04, U5 STM32F405RGTx, U6 USBLC6-2SC6, U7 TJA1051T-3, U8 R-78S3.3-0.1, U9 LP5907MFX-3.3, Y1 Crystal

Commit message: isolated drivers, layout
Parts:
- removed the C7 at (112.6, 202.5)
- removed DRV1, DRV2, DRV3: UCC21222, Package_SO:SOIC-16_3.9x9.9mm_P1.27mm
- removed the R13 at (99.9, 221.8)
- removed the R25 at (87.3, 218.1)
- removed the R26 at (87.3, 224.0)
- removed the R27 at (128.2, 183.3)
- removed the R28 at (143.3, 168.3)
- removed the R29 at (142.2, 165.4)
- removed the R30 at (125.3, 186.3)
- removed the R41 at (130.0, -29.5)
- added C1: 2.2u 35V, Capacitor_SMD:C_1206_3216Metric, F.Cu at (97.0, 22.0)
- added H10: M3, MountingHole:MountingHole_3.2mm_M3_Pad_Via, F.Cu at (63.0, -14.0)
- added H2: M3, MountingHole:MountingHole_3.2mm_M3_Pad_Via, F.Cu at (164.0, -64.0)
- added H3: M3, MountingHole:MountingHole_3.2mm_M3_Pad_Via, F.Cu at (97.0, -64.0)
- added H6: M3, MountingHole:MountingHole_3.2mm_M3_Pad_Via, F.Cu at (130.0, -15.0)
- added H8: M3, MountingHole:MountingHole_3.2mm_M3_Pad_Via, F.Cu at (197.5, -15.0)
- added R19: R, Resistor_SMD:R_0603_1608Metric, F.Cu at (71.5, 41.2)
- added R32: 200u, moje:LRMAP5930x, B.Cu at (130.0, -29.5)
- added U1: UCC21520DW, Package_SO:SOIC-16W_7.5x10.3mm_P1.27mm, B.Cu at (94.5, -20.5)
- added U3: UCC21520DW, Package_SO:SOIC-16W_7.5x10.3mm_P1.27mm, B.Cu at (164.0, -22.5)
- added U5: INA240A1D, Package_SO:SOIC-8_3.9x4.9mm_P1.27mm, F.Cu at (206.4, 29.8)
- C10, C11, C12: value 10n -> 100n; footprint Capacitor_SMD:C_0603_1608Metric -> Capacitor_SMD:C_0805_2012Metric
- C13, C14, C15: value 220n -> 10n
- C16, C17, C18: value 2.2u 35V -> 100n
- C19, C28, D1: moved to B.Cu
- C2, C3: value 10n -> 2.2u 35V; footprint Capacitor_SMD:C_0603_1608Metric -> Capacitor_SMD:C_1206_3216Metric
- C22: renamed from C25; moved to B.Cu
- C23, C24: value 10n -> 2.2u 35V; footprint Capacitor_SMD:C_0805_2012Metric -> Capacitor_SMD:C_1206_3216Metric
- C25: renamed from C22; moved to B.Cu
- C26, C27: value 2.2u 35V -> 10n; footprint Capacitor_SMD:C_1206_3216Metric -> Capacitor_SMD:C_0805_2012Metric
- J15, J16: moved to F.Cu
- Q1, Q10, Q11, Q12, Q13, Q14, Q15, Q16, Q17, Q18, Q19, Q2, Q20, Q21, Q22, Q23, Q24, Q3, Q4, Q5, Q6, Q7, Q8, Q9: footprint Package_TO_SOT_THT:TO-220-3_Horizontal_TabUp -> moje:TO-220-3_hor_tabup
- R10: renamed from R16; moved to B.Cu
- R11, R12: value R -> 2.2; footprint Resistor_SMD:R_0603_1608Metric -> Resistor_SMD:R_1206_3216Metric
- R17, R18: value 2.2 -> R; footprint Resistor_SMD:R_1206_3216Metric -> Resistor_SMD:R_0603_1608Metric
- R25: renamed from R31; value R -> 10; moved to B.Cu
- R26: renamed from R32; value R -> 10; moved to B.Cu
- R27: renamed from R33; value R -> 10; moved to B.Cu
- R28: renamed from R34; value R -> 10
- R29: renamed from R35; value R -> 10
- R30: renamed from R36; value R -> 10
- R34: renamed from R43; value R -> 10; moved to B.Cu
- R35: renamed from R44; value R -> 10
- R36: renamed from R45; value R -> 10; moved to B.Cu
- R37: renamed from R46; value R -> 10
- R38: renamed from R47; value R -> 10; moved to B.Cu
- R39: renamed from R48; value R -> 10
- R40: renamed from R49; value R -> 10; moved to B.Cu
- R41: renamed from R50; value R -> 10
- R42: renamed from R51; value R -> 10; moved to B.Cu
- R43: renamed from R52; value R -> 10
- R44: renamed from R53; value R -> 10; moved to B.Cu
- R45: renamed from R54; value R -> 10
- R46: renamed from R55; value R -> 10; moved to B.Cu
- R47: renamed from R56; value R -> 10
- R48: renamed from R57; value R -> 10; moved to B.Cu
- R49: renamed from R58; value R -> 10
- R50: renamed from R59; value R -> 10; moved to B.Cu
- R51: renamed from R60; value R -> 10
- U2: value INA240A1D -> UCC21520DW; footprint Package_SO:SOIC-8_3.9x4.9mm_P1.27mm -> Package_SO:SOIC-16W_7.5x10.3mm_P1.27mm; moved to B.Cu
- U6: renamed from U3; moved to B.Cu
- moved H4 334.3 mm to (228.5, -64.0)
- moved H1 309.9 mm to (31.0, -64.0)
- moved R44 295.9 mm to (203.0, -56.0), turned to 270 degrees
- moved H9 284.8 mm to (236.5, 3.50)
- moved R50 282.2 mm to (212.8, -55.9), turned to 270 degrees
- moved R38 280.9 mm to (182.5, -55.9), turned to 270 degrees
- moved R30 273.1 mm to (220.5, -29.5), turned to 90 degrees
- moved R46 272.2 mm to (37.0, -56.0), turned to 270 degrees
- moved R45 270.8 mm to (190.0, -29.5), turned to 90 degrees
- moved R39 269.4 mm to (210.0, -29.5), turned to 90 degrees
- moved R27 262.5 mm to (172.0, -56.0), turned to 270 degrees
- moved R48 260.0 mm to (145.2, -55.9), turned to 270 degrees
- moved R36 257.7 mm to (115.0, -56.0), turned to 270 degrees
- moved R40 256.0 mm to (47.5, -56.0), turned to 270 degrees
- moved R34 253.5 mm to (68.0, -56.0), turned to 270 degrees
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- renumbered C1 to C4, C96 to C59, C97 to C60, C98 to C61, C59 to C62, C60 to C63, C61 to C64, C62 to C65, C63 to C66, C64 to C67, C65 to C68, C66 to C69, C4 to C7, C67 to C70, C68 to C71, C69 to C72, C70 to C73, C71 to C74, C72 to C75, C73 to C76, C74 to C77, C75 to C78, C76 to C79, C77 to C80, C78 to C81, C79 to C82, C80 to C83, C81 to C84, C82 to C85, C83 to C86, C84 to C87, C85 to C88, C86 to C89, C87 to C90, C88 to C91, C89 to C92, C90 to C93, C91 to C94, C92 to C95, C93 to C96, C94 to C97, C95 to C98, H2 to H4, H3 to H7, H4 to H9, R10 to R13, R19 to R16, R40 to R31, R42 to R33, R61 to R52, R62 to R53, R63 to R54, R64 to R55, R65 to R56, R66 to R57, R67 to R58, R68 to R59, R69 to R60, R70 to R61, R71 to R62, R72 to R63, R73 to R64, R74 to R65, R75 to R66, R76 to R67, R77 to R68, R78 to R69, R79 to R70, R80 to R71, R81 to R72, R82 to R73, R83 to R74, R84 to R75, R85 to R76, R86 to R77, R87 to R78, R88 to R79, U7 to U10, U8 to U11, U9 to U12, U1 to U4, U4 to U7, U5 to U8, U6 to U9
Connections:
- net Net-(Q10-Pad3) renamed /power stage/GND_V
- net Net-(Q12-Pad3) renamed /power stage/GND_W
- net Net-(Q14-Pad3) renamed /power stage/GND_U
- C10 pad 1: GND -> +3V3
- C10 pad 2: Net-(C10-Pad2) -> GND
- C11 pad 1: GND -> +3V3
- C11 pad 2: Net-(C11-Pad2) -> GND
- C12 pad 1: GND -> +3V3
- C12 pad 2: Net-(C12-Pad2) -> GND
- C13 pad 1: +3V3 -> GND
- C13 pad 2: GND -> Net-(C13-Pad2)
- C14 pad 1: +3V3 -> GND
- C14 pad 2: GND -> Net-(C14-Pad2)
- C15 pad 1: +3V3 -> GND
- C15 pad 2: GND -> Net-(C15-Pad2)
- C16 pad 1: +3V3 -> Net-(C16-Pad1)
- C17 pad 1: +3V3 -> Net-(C17-Pad1)
- C18 pad 1: +3V3 -> Net-(C18-Pad1)
- C2 pad 1: GND -> +3V3
- C2 pad 2: Net-(C2-Pad2) -> GND
- C23 pad 1: /power stage/VBOOT_V -> +12V
- C23 pad 2: /power stage/PHASE_V -> GND
- C24 pad 1: /power stage/VBOOT_W -> +12V
- C24 pad 2: /power stage/PHASE_W -> GND
- C26 pad 1: +12V -> /power stage/VBOOT_V
- C26 pad 2: GND -> /power stage/PHASE_V
- C27 pad 1: +12V -> /power stage/VBOOT_W
- C27 pad 2: GND -> /power stage/PHASE_W
- C3 pad 1: GND -> +3V3
- C3 pad 2: Net-(C3-Pad2) -> GND
- Q1 pad 1: VDC -> Net-(Q1-Pad1)
- Q1 pad 2: Net-(Q1-Pad2) -> VDC
- Q10 pad 1: /power stage/PHASE_V -> Net-(Q10-Pad1)
- Q10 pad 2: Net-(Q10-Pad2) -> /power stage/PHASE_V
- Q11 pad 1: VDC -> Net-(Q11-Pad1)
- Q11 pad 2: Net-(Q11-Pad2) -> VDC
- Q12 pad 1: /power stage/PHASE_W -> Net-(Q12-Pad1)
- Q12 pad 2: Net-(Q12-Pad2) -> /power stage/PHASE_W
- Q13 pad 1: VDC -> Net-(Q13-Pad1)
- Q13 pad 2: Net-(Q13-Pad2) -> VDC
- Q14 pad 1: /power stage/PHASE_U -> Net-(Q14-Pad1)
- Q14 pad 2: Net-(Q14-Pad2) -> /power stage/PHASE_U
- Q15 pad 1: VDC -> Net-(Q15-Pad1)
- Q15 pad 2: Net-(Q15-Pad2) -> VDC
- Q16 pad 1: /power stage/PHASE_V -> Net-(Q16-Pad1)
- Q16 pad 2: Net-(Q16-Pad2) -> /power stage/PHASE_V
- Q17 pad 1: VDC -> Net-(Q17-Pad1)
- Q17 pad 2: Net-(Q17-Pad2) -> VDC
- Q18 pad 1: /power stage/PHASE_W -> Net-(Q18-Pad1)
- Q18 pad 2: Net-(Q18-Pad2) -> /power stage/PHASE_W
- Q19 pad 1: VDC -> Net-(Q19-Pad1)
- Q19 pad 2: Net-(Q19-Pad2) -> VDC
- Q2 pad 1: /power stage/PHASE_U -> Net-(Q2-Pad1)
- Q2 pad 2: Net-(Q2-Pad2) -> /power stage/PHASE_U
- Q20 pad 1: /power stage/PHASE_U -> Net-(Q20-Pad1)
- Q20 pad 2: Net-(Q20-Pad2) -> /power stage/PHASE_U
- Q21 pad 1: VDC -> Net-(Q21-Pad1)
- Q21 pad 2: Net-(Q21-Pad2) -> VDC
- Q22 pad 1: /power stage/PHASE_V -> Net-(Q22-Pad1)
- Q22 pad 2: Net-(Q22-Pad2) -> /power stage/PHASE_V
- Q23 pad 1: VDC -> Net-(Q23-Pad1)
- Q23 pad 2: Net-(Q23-Pad2) -> VDC
- Q24 pad 1: /power stage/PHASE_W -> Net-(Q24-Pad1)
- Q24 pad 2: Net-(Q24-Pad2) -> /power stage/PHASE_W
- Q3 pad 1: VDC -> Net-(Q3-Pad1)
- Q3 pad 2: Net-(Q3-Pad2) -> VDC
- Q4 pad 1: /power stage/PHASE_V -> Net-(Q4-Pad1)
- Q4 pad 2: Net-(Q4-Pad2) -> /power stage/PHASE_V
- Q5 pad 1: VDC -> Net-(Q5-Pad1)
- Q5 pad 2: Net-(Q5-Pad2) -> VDC
- Q6 pad 1: /power stage/PHASE_W -> Net-(Q6-Pad1)
- Q6 pad 2: Net-(Q6-Pad2) -> /power stage/PHASE_W
- Q7 pad 1: VDC -> Net-(Q7-Pad1)
- Q7 pad 2: Net-(Q7-Pad2) -> VDC
- Q8 pad 1: /power stage/PHASE_U -> Net-(Q8-Pad1)
- Q8 pad 2: Net-(Q8-Pad2) -> /power stage/PHASE_U
- Q9 pad 1: VDC -> Net-(Q9-Pad1)
- Q9 pad 2: Net-(Q9-Pad2) -> VDC
- R11 pad 1: Net-(C2-Pad2) -> Net-(D2-Pad2)
- R11 pad 2: GND -> +12V
- R12 pad 1: Net-(C3-Pad2) -> Net-(D3-Pad2)
- R12 pad 2: GND -> +12V
- R14 pad 1: GND -> Net-(C5-Pad2)
- R14 pad 2: Net-(C11-Pad2) -> GND
- R15 pad 1: GND -> Net-(C6-Pad2)
- R15 pad 2: Net-(C12-Pad2) -> GND
- R17 pad 1: Net-(D2-Pad2) -> Net-(C8-Pad2)
- R17 pad 2: +12V -> GND
- R18 pad 1: Net-(D3-Pad2) -> Net-(C9-Pad2)
- R18 pad 2: +12V -> GND
- R20 pad 1: Net-(C5-Pad2) -> GND
- R20 pad 2: GND -> Net-(C17-Pad1)
- R21 pad 1: Net-(C6-Pad2) -> GND
- R21 pad 2: GND -> Net-(C18-Pad1)
- R22 pad 1: Net-(C7-Pad2) (its old number) -> Net-(C13-Pad2)
- R23 pad 1: Net-(C8-Pad2) -> Net-(C14-Pad2)
- R24 pad 1: Net-(C9-Pad2) -> Net-(C15-Pad2)
- R25 pad 2: Net-(Q1-Pad2) -> Net-(Q1-Pad1)
- R26 pad 1: Net-(R27-Pad2) -> Net-(R26-Pad1)
- R26 pad 2: Net-(Q3-Pad2) -> Net-(Q3-Pad1)
- R27 pad 2: Net-(Q5-Pad2) -> Net-(Q5-Pad1)
- R28 pad 2: Net-(Q2-Pad2) -> Net-(Q2-Pad1)
- R29 pad 1: Net-(R28-Pad1) (its old number) -> Net-(R29-Pad1)
- R29 pad 2: Net-(Q4-Pad2) -> Net-(Q4-Pad1)
- R3 pad 1: Net-(C7-Pad2) (its old number) -> Net-(C13-Pad2)
- R30 pad 2: Net-(Q6-Pad2) -> Net-(Q6-Pad1)
- R34 pad 2: Net-(Q7-Pad2) -> Net-(Q7-Pad1)
- R35 pad 2: Net-(Q8-Pad2) -> Net-(Q8-Pad1)
- R36 pad 1: Net-(R27-Pad2) -> Net-(R26-Pad1)
- R36 pad 2: Net-(Q9-Pad2) -> Net-(Q9-Pad1)
- R37 pad 1: Net-(R28-Pad1) (its old number) -> Net-(R29-Pad1)
- R37 pad 2: Net-(Q10-Pad2) -> Net-(Q10-Pad1)
- R38 pad 2: Net-(Q11-Pad2) -> Net-(Q11-Pad1)
- R39 pad 2: Net-(Q12-Pad2) -> Net-(Q12-Pad1)
- R4 pad 1: Net-(C2-Pad2) -> Net-(C5-Pad2)
- R40 pad 2: Net-(Q13-Pad2) -> Net-(Q13-Pad1)
- R41 pad 2: Net-(Q14-Pad2) -> Net-(Q14-Pad1)
- R42 pad 1: Net-(R27-Pad2) -> Net-(R26-Pad1)
- R42 pad 2: Net-(Q15-Pad2) -> Net-(Q15-Pad1)
- R43 pad 1: Net-(R28-Pad1) (its old number) -> Net-(R29-Pad1)
- R43 pad 2: Net-(Q16-Pad2) -> Net-(Q16-Pad1)
- R44 pad 2: Net-(Q17-Pad2) -> Net-(Q17-Pad1)
- R45 pad 2: Net-(Q18-Pad2) -> Net-(Q18-Pad1)
- R46 pad 2: Net-(Q19-Pad2) -> Net-(Q19-Pad1)
- R47 pad 2: Net-(Q20-Pad2) -> Net-(Q20-Pad1)
- R48 pad 1: Net-(R27-Pad2) -> Net-(R26-Pad1)
- R48 pad 2: Net-(Q21-Pad2) -> Net-(Q21-Pad1)
- R49 pad 1: Net-(R28-Pad1) (its old number) -> Net-(R29-Pad1)
- R49 pad 2: Net-(Q22-Pad2) -> Net-(Q22-Pad1)
- R5 pad 1: Net-(C5-Pad2) -> Net-(C8-Pad2)
- R50 pad 2: Net-(Q23-Pad2) -> Net-(Q23-Pad1)
- R51 pad 2: Net-(Q24-Pad2) -> Net-(Q24-Pad1)
- R6 pad 1: Net-(C8-Pad2) -> Net-(C14-Pad2)
- R7 pad 1: Net-(C3-Pad2) -> Net-(C6-Pad2)
- R8 pad 1: Net-(C6-Pad2) -> Net-(C9-Pad2)
- R9 pad 1: Net-(C9-Pad2) -> Net-(C15-Pad2)
- U2 pad 1: Net-(R41-Pad3) -> Net-(C5-Pad2)
- U2 pad 2: GNDA -> Net-(C8-Pad2)
- U2 pad 3: GNDA -> +3V3
- U2 pad 4: GNDA -> GND
- U2 pad 5: /mcu/ISENSE_V -> Net-(C14-Pad2)
- U2 pad 6: Net-(C32-Pad1) -> Net-(C17-Pad1)
- U2 pad 7: +3V3 -> Net-(U2-Pad7)
- U2 pad 8: Net-(R41-Pad2) -> +3V3
Routing:
- net Net-(R25-Pad1): track 0.00 -> 89.2 mm, vias 0 -> 1
- net Net-(R26-Pad1): track 0.00 -> 76.7 mm, vias 0 -> 1
- net Net-(R27-Pad1): track 0.00 -> 64.4 mm, vias 0 -> 1
- net Net-(R28-Pad1): track 0.00 -> 49.8 mm
- net Net-(R31-Pad3): track 0.00 -> 5.40 mm, vias 0 -> 1
- net Net-(Q13-Pad1): track 0.00 -> 3.14 mm
- net Net-(R31-Pad2): track 0.00 -> 2.75 mm
- net Net-(Q23-Pad1): track 0.00 -> 2.75 mm
- net Net-(Q21-Pad1): track 0.00 -> 2.75 mm
- net Net-(Q19-Pad1): track 0.00 -> 2.68 mm
- net Net-(Q8-Pad1): track 0.00 -> 2.62 mm
- net Net-(Q2-Pad1): track 0.00 -> 2.61 mm
- net Net-(Q20-Pad1): track 0.00 -> 2.56 mm
- net Net-(Q14-Pad1): track 0.00 -> 2.56 mm
- net Net-(Q1-Pad1): track 0.00 -> 2.53 mm
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- added copper zone on B.Cu, net /power stage/GND_U
- added copper zone on In1.Cu, net /power stage/GND_U
- added copper zone on In2.Cu, net /power stage/GND_U
- added copper zone on B.Cu, net /power stage/GND_V
- added copper zone on In1.Cu, net /power stage/GND_V
- added copper zone on In2.Cu, net /power stage/GND_V
- added copper zone on B.Cu, net /power stage/GND_W
- added copper zone on In1.Cu, net /power stage/GND_W
- added copper zone on In2.Cu, net /power stage/GND_W
- added copper zone on F.Cu, net /power stage/PHASE_U
- added copper zone on In1.Cu, net /power stage/PHASE_U
- added copper zone on In2.Cu, net /power stage/PHASE_U
- added copper zone on F.Cu, net /power stage/PHASE_V
- added copper zone on In1.Cu, net /power stage/PHASE_V
- added copper zone on In2.Cu, net /power stage/PHASE_V
- added copper zone on F.Cu, net /power stage/PHASE_W
- added copper zone on In1.Cu, net /power stage/PHASE_W
- added copper zone on In2.Cu, net /power stage/PHASE_W
- added copper zone on B.Cu, net GND
- added copper zone on F.Cu, net GND
- added copper zone on In1.Cu, net GND
- added copper zone on In2.Cu, net GND
- added copper zone on B.Cu, net VDC
- added copper zone on F.Cu, net VDC
- added copper zone on In1.Cu, net VDC
- added copper zone on In2.Cu, net VDC
Other:
- board size 230 x 45 mm -> 231 x 75 mm
- copper layers 2 -> 4

Commit message: 12V PS, isolated gate drivers
Parts:
- added C100: 0.47u 200V, Capacitor_SMD:C_0603_1608Metric, F.Cu at (10.0, 24.5)
- added C101: 0.47u 200V, Capacitor_SMD:C_0603_1608Metric, F.Cu at (11.3, 38.3)
- added C102: 0.47u 200V, Capacitor_SMD:C_0603_1608Metric, F.Cu at (10.0, 27.1)
- added C103: 100n, Capacitor_SMD:C_0603_1608Metric, F.Cu at (11.3, 40.8)
- added C104: 4.7u, Capacitor_SMD:C_0603_1608Metric, F.Cu at (14.0, 24.5)
- added C105: 4.7u, Capacitor_SMD:C_0603_1608Metric, F.Cu at (15.3, 38.3)
- added C106: 4.7u, Capacitor_SMD:C_0603_1608Metric, F.Cu at (10.0, 29.6)
- added C107: 4.7u, Capacitor_SMD:C_0603_1608Metric, F.Cu at (14.0, 27.1)
- added C108: 4.7u, Capacitor_SMD:C_0603_1608Metric, F.Cu at (15.3, 40.8)
- added C112: 1n, Capacitor_SMD:C_0603_1608Metric, F.Cu at (13.0, 43.3)
- added C113: 10p, Capacitor_SMD:C_0603_1608Metric, F.Cu at (19.3, 38.3)
- added C114: 0.1u, Capacitor_SMD:C_0603_1608Metric, F.Cu at (14.0, 29.6)
- added C115: 2.2u, Capacitor_SMD:C_0603_1608Metric, F.Cu at (18.0, 24.8)
- added C116: 100p, Capacitor_SMD:C_0603_1608Metric, F.Cu at (19.3, 40.8)
- added C117: 4.7n, Capacitor_SMD:C_0603_1608Metric, F.Cu at (17.0, 43.3)
- added H6: M3, MountingHole:MountingHole_3.2mm_M3_Pad_Via, F.Cu at (-10.5, 3.50)
- added IC1: LTC7801, Package_DFN_QFN:QFN-24-1EP_4x5mm_P0.5mm_EP2.65x3.65mm, F.Cu at (19.5, 32.5)
- added R80: 8m, Resistor_SMD:R_0603_1608Metric, F.Cu at (23.3, 38.3)
- added R81: 100k, Resistor_SMD:R_0603_1608Metric, F.Cu at (18.0, 27.3)
- added R82: 511k, Resistor_SMD:R_0603_1608Metric, F.Cu at (22.0, 24.8)
- added R83: 10p, Resistor_SMD:R_0603_1608Metric, F.Cu at (23.3, 40.8)
- added R84: 10k, Resistor_SMD:R_0603_1608Metric, F.Cu at (21.0, 43.3)
- added R85: 80k6, Resistor_SMD:R_0603_1608Metric, F.Cu at (27.3, 38.3)
- added R86: 30k1, Resistor_SMD:R_0603_1608Metric, F.Cu at (22.0, 27.3)
- C1: renamed from C19; value 2.2u 35V -> 4.7u 25V
- C23: renamed from C16; footprint Capacitor_SMD:C_0805_2012Metric -> Capacitor_SMD:C_0603_1608Metric
- C24: renamed from C1; moved to B.Cu
- C25: renamed from C10; moved to B.Cu
- C36: renamed from C20; value 2.2u 35V -> 4.7u 25V; moved to B.Cu
- C37: renamed from C26; moved to B.Cu
- C41: renamed from C17; footprint Capacitor_SMD:C_0805_2012Metric -> Capacitor_SMD:C_0603_1608Metric
- C44: renamed from C23; value 2.2u 35V -> 4.7u 25V; moved to B.Cu
- C45: renamed from C29; moved to B.Cu
- C49: renamed from C21; value 2.2u 35V -> 4.7u 25V; moved to B.Cu
- C50: renamed from C27; moved to B.Cu
- C54: renamed from C18; footprint Capacitor_SMD:C_0805_2012Metric -> Capacitor_SMD:C_0603_1608Metric
- C57: renamed from C24; value 2.2u 35V -> 4.7u 25V; moved to B.Cu
- C58: renamed from C30; moved to B.Cu
- D2, D3: moved to B.Cu
- J16: value 12V IN -> 12V OUT
- R10: renamed from R52; footprint Resistor_SMD:R_1210_3225Metric -> Resistor_SMD:R_0805_2012Metric
- R20: renamed from R11; moved to B.Cu
- R29: renamed from R54; footprint Resistor_SMD:R_1210_3225Metric -> Resistor_SMD:R_0805_2012Metric
- R39: renamed from R12; moved to B.Cu
- R51: renamed from R56; footprint Resistor_SMD:R_1210_3225Metric -> Resistor_SMD:R_0805_2012Metric
- U6: moved to F.Cu
- moved C57 155.0 mm to (226.0, -29.5), turned to 180 degrees
- moved C58 150.7 mm to (226.0, -27.0), turned to 180 degrees
- moved D3 146.4 mm to (237.5, -27.0), turned to 270 degrees
- moved C50 141.5 mm to (232.5, -27.0), turned to 180 degrees
- moved C49 139.7 mm to (232.5, -29.5), turned to 180 degrees
- moved R39 137.6 mm to (237.5, -20.0), turned to 270 degrees
- moved U3 131.5 mm to (162.0, -21.0)
- moved U10 129.4 mm to (148.5, 18.5), turned to 90 degrees
- moved C44 102.9 mm to (159.0, -30.5), turned to 180 degrees
- moved D2 101.8 mm to (169.5, -28.0), turned to 270 degrees
- moved C36 98.8 mm to (165.0, -30.5), turned to 180 degrees
- moved C15 96.6 mm to (95.0, -18.0), turned to 270 degrees
- moved U4 94.1 mm to (129.5, -24.5)
- moved C45 92.0 mm to (159.0, -28.0), turned to 180 degrees
- moved C14 89.8 mm to (99.0, -18.0), turned to 270 degrees
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- renumbered C58 to C10, C59 to C11, C60 to C12, C61 to C13, C4 to C14, C7 to C15, C13 to C16, C41 to C17, C44 to C18, C47 to C19, C25 to C2, C50 to C20, C53 to C21, C55 to C22, C22 to C26, C28 to C27, C31 to C28, C34 to C29, C40 to C3, C37 to C30, C42 to C31, C45 to C32, C48 to C33, C51 to C34, C54 to C35, C5 to C38, C8 to C39, C43 to C4, C14 to C40, C2 to C42, C11 to C43, C32 to C46, C35 to C47, C38 to C48, C46 to C5, C6 to C51, C9 to C52, C15 to C53, C3 to C55, C12 to C56, C33 to C59, C49 to C6, C36 to C60, C39 to C61, C64 to C63, C68 to C64, C69 to C65, C70 to C66, C71 to C67, C75 to C68, C77 to C69, C52 to C7, C79 to C70, C80 to C71, C81 to C72, C82 to C73, C83 to C74, C74 to C75, C65 to C76, C76 to C77, C66 to C79, C56 to C8, C72 to C80, C73 to C81, C67 to C82, C63 to C83, C89 to C84, C90 to C85, C84 to C86, C85 to C87, C91 to C88, C86 to C89, C57 to C9, C87 to C90, C88 to C91, C95 to C94, C94 to C95, FB4 to FB3, FB5 to FB4, FB3 to FB5, H6 to H10, H4 to H2, H7 to H3, H9 to H4, H2 to H5, H8 to H7, H10 to H8, H3 to H9, J15 to J10, J9 to J11, J11 to J12, J12 to J15, J4 to J2, J5 to J3, J2 to J4, J6 to J5, J7 to J6, J3 to J7, J10 to J9, Q9 to Q10, Q15 to Q11, Q21 to Q12, Q4 to Q13, Q10 to Q14, Q16 to Q15, Q22 to Q16, Q5 to Q17, Q11 to Q18, Q17 to Q19, Q7 to Q2, Q23 to Q20, Q6 to Q21, Q12 to Q22, Q18 to Q23, Q13 to Q3, Q19 to Q4, Q2 to Q5, Q8 to Q6, Q14 to Q7, Q20 to Q8, Q3 to Q9, R10 to R1, R2 to R11, R28 to R12, R35 to R13, R41 to R14, R47 to R15, R3 to R16, R53 to R17, R19 to R18, R31 to R19, R25 to R2, R26 to R21, R36 to R22, R42 to R23, R48 to R24, R14 to R25, R17 to R26, R23 to R27, R4 to R28, R34 to R3, R5 to R30, R29 to R31, R37 to R32, R43 to R33, R49 to R34, R6 to R35, R55 to R36, R20 to R37, R32 to R38, R40 to R4, R59 to R40, R27 to R41, R38 to R42, R44 to R43, R50 to R44, R60 to R45, R15 to R46, R18 to R47, R24 to R48, R58 to R49, R46 to R5, R7 to R50, R8 to R52, R30 to R53, R39 to R54, R45 to R55, R51 to R56, R9 to R57, R57 to R58, R21 to R59, R13 to R6, R33 to R60, R64 to R61, R61 to R62, R62 to R63, R63 to R64, R72 to R68, R73 to R69, R16 to R7, R78 to R70, R79 to R71, R68 to R72, R69 to R73, R70 to R74, R71 to R76, R74 to R77, R76 to R78, R77 to R79, R22 to R8, R1 to R9, U4 to U2, U2 to U3, U5 to U4, U3 to U5, U8 to U7, U7 to U8
Routing:
- net Net-(R2-Pad1): track 89.2 -> 103.9 mm, vias 1 -> 2
- net Net-(R12-Pad1): track 49.8 -> 59.2 mm, vias 0 -> 1
- net +12V: track 0.00 -> 4.98 mm
- net GND: track 0.00 -> 4.87 mm
- net Net-(R19-Pad2): track 2.75 -> 0.00 mm
- net /power stage/PHASE_U: vias 0 -> 5
- net /power stage/GND_W: vias 0 -> 70
- net (no net): vias 70 -> 0
- added copper zone on B.Cu, net /power stage/PHASE_U

Commit message: layout and routing progress
Parts:
- removed the C100 at (10.0, 24.5)
- removed the C103 at (11.3, 40.8)
- removed the C106 at (10.0, 29.6)
- removed C113: 10p, Capacitor_SMD:C_0603_1608Metric
- removed the C35 at (168.7, 28.8)
- removed C95: 100u, Capacitor_Tantalum_SMD:CP_EIA-6032-28_Kemet-C
- removed the FB3 at (134.0, 34.0)
- removed FB4: FB, Inductor_SMD:L_0603_1608Metric
- removed the H6 at (-10.5, 3.50)
- removed NT1, NT2, NT3: nt, NetTie:NetTie-2_THT_Pad1.0mm
- removed the Q13 at (153.0, -33.0)
- removed the R80 at (23.3, 38.3)
- removed the R81 at (18.0, 27.3)
- removed the R82 at (22.0, 24.8)
- removed the R83 at (23.3, 40.8)
- removed the R86 at (22.0, 27.3)
- added C110: 4.7u 25V, Capacitor_SMD:C_1206_3216Metric, F.Cu at (30.0, -14.2)
- added C111: 4.7u 25V, Capacitor_SMD:C_1206_3216Metric, F.Cu at (30.0, -11.5)
- added C54: 2.2u, Capacitor_SMD:C_0603_1608Metric, F.Cu at (153.0, -18.5)
- added C93: 0.47u 200V, Capacitor_SMD:C_1206_3216Metric, F.Cu at (24.0, -14.2)
- added C94: 0.47u 200V, Capacitor_SMD:C_1206_3216Metric, F.Cu at (24.0, -9.25)
- added C96: 100n, Capacitor_SMD:C_0603_1608Metric, F.Cu at (18.2, -13.5)
- added C98: 0.47u 200V, Capacitor_SMD:C_1206_3216Metric, B.Cu at (20.2, -19.8)
- added C99: 4.7u, Capacitor_SMD:C_0603_1608Metric, F.Cu at (19.5, -20.2)
- added D7: ESD 100V, Diode_SMD:D_SOD-123, B.Cu at (18.8, -4.50)
- added D8: LED, LED_SMD:LED_0603_1608Metric, F.Cu at (11.0, -13.5)
- added D9: 12.7, Diode_SMD:D_SMA, B.Cu at (38.5, -5.65)
- added J15: IGNITION, Connector_PinHeader_2.54mm:PinHeader_1x02_P2.54mm_Vertical, F.Cu at (24.0, -2.62)
- added L1: 7443633300, moje:WE-HCF-2013, F.Cu at (45.0, -15.2)
- added Q25: FDMS86252L, moje:TDSON-8-MOS, F.Cu at (24.2, -19.5)
- added Q26: BSC110N15NS5, moje:TDSON-8-MOS, F.Cu at (30.5, -19.5)
- added Q4: Q_NMOS_DGS, moje:TO-220-3_hor_tabup, B.Cu at (153.0, -33.0)
- added R58: 1R, Resistor_SMD:R_1206_3216Metric, B.Cu at (26.0, -44.0)
- added R59: 1R, Resistor_SMD:R_1206_3216Metric, B.Cu at (227.5, -44.0)
- added R61: 1R, Resistor_SMD:R_1206_3216Metric, B.Cu at (161.5, -44.0)
- added R62: 1R, Resistor_SMD:R_1206_3216Metric, B.Cu at (93.8, -44.0)
- added R87: 470, Resistor_SMD:R_0603_1608Metric, F.Cu at (11.0, -10.2)
- added R88: 1M, Resistor_SMD:R_0603_1608Metric, F.Cu at (15.2, -13.5)
- added R89: 9k1, Resistor_SMD:R_0603_1608Metric, F.Cu at (16.8, -13.5)
- added R90: 100k, Resistor_SMD:R_0603_1608Metric, F.Cu at (12.8, -13.5)
- added R91: 80k6, Resistor_SMD:R_0603_1608Metric, B.Cu at (15.2, -23.8)
- added R92: 10k, Resistor_SMD:R_0603_1608Metric, F.Cu at (19.5, -17.8)
- added R93: 10R, Resistor_SMD:R_0603_1608Metric, B.Cu at (20.2, -15.8)
- added R94: 30k1, Resistor_SMD:R_0603_1608Metric, B.Cu at (13.5, -23.8)
- added R95: 71.5k, Resistor_SMD:R_0603_1608Metric, F.Cu at (11.8, -18.2)
- added R96: 80k6, Resistor_SMD:R_0603_1608Metric, B.Cu at (18.8, -13.5)
- added R97: 255k, Resistor_SMD:R_0603_1608Metric, B.Cu at (16.5, -12.8)
- added R98: 60k4, Resistor_SMD:R_0603_1608Metric, B.Cu at (11.8, -12.8)
- added R99: 4k32, Resistor_SMD:R_0603_1608Metric, B.Cu at (11.8, -16.2)
- C100: renamed from C94; value 2.2u -> 4.7u; footprint Capacitor_SMD:C_0603_1608Metric -> Capacitor_SMD:C_1206_3216Metric; moved to B.Cu
- C101: value 0.47u 200V -> 100n 50V; moved to B.Cu
- C102: value 0.47u 200V -> 2.2u 10V; moved to B.Cu
- C104: value 4.7u -> 270p
- C105: value 4.7u -> 130p
- C107: value 4.7u -> 47n; moved to B.Cu
- C108: value 4.7u -> 10p; moved to B.Cu
- C11: renamed from C43; moved to B.Cu
- C112: value 1n -> 4.7u 25V; footprint Capacitor_SMD:C_0603_1608Metric -> Capacitor_SMD:C_1206_3216Metric
- C114: value 0.1u -> 4.7u 25V; footprint Capacitor_SMD:C_0603_1608Metric -> Capacitor_SMD:C_1206_3216Metric
- C115: value 2.2u -> TR3D157K016C0075; footprint Capacitor_SMD:C_0603_1608Metric -> Capacitor_Tantalum_SMD:CP_EIA-7343-31_Kemet-D; moved to B.Cu
- C116: value 100p -> TR3D157K016C0075; footprint Capacitor_SMD:C_0603_1608Metric -> Capacitor_Tantalum_SMD:CP_EIA-7343-31_Kemet-D; moved to B.Cu
- C117: value 4.7n -> TR3D157K016C0075; footprint Capacitor_SMD:C_0603_1608Metric -> Capacitor_Tantalum_SMD:CP_EIA-7343-31_Kemet-D; moved to B.Cu
- C12: renamed from C56; moved to B.Cu
- C2: renamed from C42; moved to B.Cu
- C3: renamed from C55; moved to B.Cu
- C40: renamed from C3; value CP -> B41858C9477M000
- C41: renamed from C17; value 22u -> F611BY685K100A
- C42: renamed from C31; value 10n -> C1206C105K1RACTU; moved to B.Cu
- C43: renamed from C4; value CP -> B41858C9477M000
- C44: renamed from C18; value 22u -> F611BY685K100A
- C45: renamed from C32; value 10n -> C1206C105K1RACTU; moved to B.Cu
- C46: renamed from C5; value CP -> B41858C9477M000
- C47: renamed from C19; value 22u -> F611BY685K100A
- C48: renamed from C33; value 10n -> C1206C105K1RACTU; moved to B.Cu
- C49: renamed from C6; value CP -> B41858C9477M000
- C50: renamed from C20; value 22u -> F611BY685K100A
- C51: renamed from C34; value 10n -> C1206C105K1RACTU; moved to B.Cu
- C52: renamed from C7; value CP -> B41858C9477M000
- C53: renamed from C21; value 22u -> F611BY685K100A
- C55: renamed from C22; value 22u -> F611BY685K100A
- C56: renamed from C8; value CP -> B41858C9477M000
- C57: renamed from C9; value CP -> B41858C9477M000
- C58: renamed from C10; value CP -> B41858C9477M000
- C59: renamed from C11; value CP -> B41858C9477M000
- C60: renamed from C12; value CP -> B41858C9477M000
- C61: renamed from C13; value CP -> B41858C9477M000
- C63: renamed from C83; value C_Small -> 100n
- C92: value 2.2u -> 0.47u 200V; footprint Capacitor_SMD:C_0603_1608Metric -> Capacitor_SMD:C_1206_3216Metric
- C97: renamed from C93; moved to B.Cu
- FB8, IC1, R84: moved to B.Cu
- J10: renamed from J9; footprint Connector_USB:USB_Micro-B_Molex_47346-0001 -> Connector_USB:USB_Micro-B_Wuerth_614105150721_Vertical_CircularHoles
- J11: renamed from J12; footprint Connector_PinHeader_2.54mm:PinHeader_1x03_P2.54mm_Vertical_SMD_Pin1Right -> Connector_PinHeader_2.54mm:PinHeader_1x03_P2.54mm_Vertical
- J17: renamed from J16; footprint Connector_PinHeader_2.54mm:PinHeader_1x02_P2.54mm_Vertical -> conn-amass:AMASS_XT30U-M_1x02_P5.0mm_Vertical
- R52: renamed from R10; value R -> 150k
- R53: renamed from R17; value R -> 3k24
- R54: renamed from R29; value R -> 150k
- R55: renamed from R36; value R -> 3k24
- R56: renamed from R51; value R -> 150k
- R57: renamed from R58; value R -> 3k24
- R60: renamed from R49; value R -> 10k; footprint Resistor_SMD:R_0805_2012Metric -> Resistor_SMD:R_0603_1608Metric
- R63: renamed from R40; value R -> 150k; footprint Resistor_SMD:R_1210_3225Metric -> Resistor_SMD:R_0805_2012Metric
- R64: renamed from R45; value R -> 3k24
- R85: value 80k6 -> 10k; moved to B.Cu
- TH1: value NTC -> 10k; moved to B.Cu
- U11: value R-78S3.3-0.1 -> R-78E5.0-0.5; footprint Converter_DCDC:Converter_DCDC_RECOM_R-78S-0.1_THT -> Converter_DCDC:Converter_DCDC_RECOM_R-78E-0.5_THT
- Y1: value Crystal -> MCSJK-7I-8.00-18-10-60-B-10
- moved C45 186.6 mm to (233.0, -44.0), turned to 180 degrees
- moved J8 175.0 mm to (164.5, -3.00), turned to 90 degrees
- moved R15 167.8 mm to (232.5, -18.0), turned to 90 degrees
- moved C3 154.0 mm to (231.0, -10.5), turned to 180 degrees
- moved C48 152.6 mm to (167.0, -44.0), turned to 180 degrees
- moved R7 150.1 mm to (233.5, -15.2)
- moved C92 149.9 mm to (24.0, -11.8)
- moved C78 149.0 mm to (139.4, 17.6)
- moved C80 149.0 mm to (154.3, 19.7)
- moved C83 149.0 mm to (162.6, 16.4)
- moved R73 149.0 mm to (158.3, 19.7)
- moved C79 149.0 mm to (153.3, 12.5)
- moved R57 145.1 mm to (237.2, -18.0), turned to 90 degrees
- moved R76 143.5 mm to (98.5, -11.0), turned to 90 degrees
- moved C12 143.1 mm to (231.0, -12.8), turned to 180 degrees
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- renumbered C24 to C1, C25 to C10, C96 to C103, C97 to C106, C98 to C109, C16 to C13, C40 to C14, C53 to C15, C23 to C16, C41 to C17, C54 to C18, C1 to C19, C36 to C20, C49 to C21, C26 to C22, C44 to C23, C57 to C24, C2 to C25, C37 to C26, C50 to C27, C27 to C28, C45 to C29, C58 to C30, C28 to C31, C46 to C32, C59 to C33, C29 to C34, C47 to C35, C60 to C36, C30 to C37, C48 to C38, C61 to C39, C14 to C4, C38 to C5, C51 to C6, C63 to C64, C76 to C65, C79 to C66, C82 to C67, C64 to C68, C65 to C69, C15 to C7, C66 to C70, C67 to C71, C80 to C72, C81 to C73, C75 to C74, C68 to C75, C77 to C76, C69 to C77, C70 to C79, C39 to C8, C71 to C80, C72 to C81, C73 to C82, C74 to C83, C86 to C84, C87 to C85, C89 to C86, C90 to C87, C91 to C88, C84 to C89, C52 to C9, C85 to C90, C88 to C91, FB5 to FB3, H5 to H2, H2 to H3, H9 to H4, H7 to H5, H10 to H6, H3 to H7, H4 to H9, J15 to J12, J10 to J16, J4 to J2, J7 to J3, J2 to J4, J3 to J5, J5 to J6, J6 to J7, J11 to J9, Q14 to Q10, Q18 to Q11, Q22 to Q12, Q3 to Q13, Q7 to Q14, Q11 to Q15, Q15 to Q16, Q19 to Q17, Q23 to Q18, Q4 to Q19, Q5 to Q2, Q8 to Q20, Q12 to Q21, Q16 to Q22, Q20 to Q23, Q9 to Q3, Q17 to Q5, Q21 to Q6, Q2 to Q7, Q6 to Q8, Q10 to Q9, R9 to R1, R1 to R10, R20 to R11, R39 to R12, R6 to R13, R25 to R14, R46 to R15, R7 to R16, R26 to R17, R47 to R18, R18 to R19, R11 to R2, R37 to R20, R59 to R21, R8 to R22, R27 to R23, R48 to R24, R2 to R25, R21 to R26, R41 to R27, R12 to R28, R31 to R29, R16 to R3, R53 to R30, R19 to R31, R38 to R32, R60 to R33, R3 to R34, R13 to R35, R22 to R36, R32 to R37, R42 to R38, R54 to R39, R28 to R4, R4 to R40, R14 to R41, R23 to R42, R33 to R43, R43 to R44, R55 to R45, R5 to R46, R15 to R47, R24 to R48, R34 to R49, R30 to R5, R44 to R50, R56 to R51, R35 to R6, R62 to R66, R63 to R67, R64 to R68, R61 to R69, R50 to R7, R65 to R70, R66 to R71, R67 to R72, R72 to R73, R73 to R74, R74 to R75, R68 to R77, R69 to R78, R77 to R79, R52 to R8, R75 to R80, R78 to R81, R79 to R82, R70 to R83, R71 to R86, R57 to R9, U3 to U2, U5 to U3, U2 to U4, U4 to U5, U8 to U7, U7 to U8
Connections:
- C100 pad 1: Net-(C93-Pad1) -> Net-(C100-Pad1)
- C101 pad 1: VDC -> /pwr mng/SW
- C101 pad 2: GND -> Net-(C101-Pad2)
- C102 pad 1: VDC -> /pwr mng/SS
- C104 pad 1: Net-(C104-Pad1) -> /pwr mng/ITH
- C105 pad 1: +12V -> Net-(C105-Pad1)
- C107 pad 1: +12V -> /pwr mng/SENSE+
- C107 pad 2: GND -> +12V
- C108 pad 2: GND -> /pwr mng/VFB
- C112 pad 1: /pwr mng/SENSE+ -> +12V
- C112 pad 2: +12V -> GND
- C114 pad 1: Net-(C114-Pad1) -> +12V
- C115 pad 1: Net-(C115-Pad1) -> +12V
- C116 pad 1: Net-(C116-Pad1) -> +12V
- C117 pad 1: Net-(C117-Pad1) -> +12V
- C31 pad 1: Net-(C28-Pad1) -> /power stage/VSUPA_U
- C32 pad 1: Net-(C46-Pad1) -> /power stage/VSUPA_V
- C33 pad 1: Net-(C59-Pad1) -> /power stage/VSUPA_W
- C34 pad 1: Net-(C28-Pad1) -> /power stage/VSUPA_U
- C35 pad 1: Net-(C46-Pad1) -> /power stage/VSUPA_V
- C36 pad 1: Net-(C59-Pad1) -> /power stage/VSUPA_W
- C42 pad 2: GND -> Net-(C42-Pad2)
- C45 pad 2: GND -> Net-(C45-Pad2)
- C48 pad 2: GND -> Net-(C48-Pad2)
- C51 pad 2: GND -> Net-(C51-Pad2)
- C92 pad 1: +12V -> VDC
- C97 pad 1: Net-(C93-Pad1) -> Net-(C100-Pad1)
- FB1 pad 2: Net-(C28-Pad1) -> /power stage/VSUPA_U
- FB2 pad 2: Net-(C46-Pad1) -> /power stage/VSUPA_V
- FB3 pad 2: Net-(C59-Pad1) -> /power stage/VSUPA_W
- FB8 pad 1: Net-(C93-Pad1) -> Net-(C100-Pad1)
- H5 pad 1: GNDS -> Net-(H5-Pad1)
- H6 pad 1: GNDS -> Net-(H6-Pad1)
- H8 pad 1: GNDS -> Net-(H8-Pad1)
- IC1 pad 1: Net-(C113-Pad2) -> /pwr mng/VFB
- IC1 pad 11: Net-(IC1-Pad11) -> /pwr mng/TOP_GATE
- IC1 pad 12: Net-(C103-Pad1) -> /pwr mng/SW
- IC1 pad 13: Net-(C103-Pad2) -> Net-(C101-Pad2)
- IC1 pad 14: Net-(IC1-Pad14) -> /pwr mng/BOTTOM_GATE
- IC1 pad 15: Net-(C104-Pad1) -> Net-(C99-Pad1)
- IC1 pad 16: Net-(C104-Pad1) -> Net-(C99-Pad1)
- IC1 pad 17: VDC -> /pwr mng/VIN+
- IC1 pad 19: /pwr mng/RUN -> /io/IGNITION
- IC1 pad 2: Net-(C116-Pad1) -> /pwr mng/ITH
- IC1 pad 20: Net-(C114-Pad1) -> /pwr mng/INTVCC
- IC1 pad 21: GND -> /pwr mng/OVLO
- IC1 pad 24: Net-(C115-Pad1) -> /pwr mng/SS
- IC1 pad 5: Net-(C114-Pad1) -> /pwr mng/INTVCC
- IC1 pad 8: Net-(IC1-Pad8) -> /pwr mng/FREQ
- IC1 pad 9: Net-(IC1-Pad9) -> /pwr mng/DRVSET
- J10 pad 4: Net-(J9-Pad4) -> (no net)
- R53 pad 1: GND -> GNDA
- R55 pad 1: GND -> GNDA
- R57 pad 1: GND -> GNDA
- R60 pad 2: Net-(FB4-Pad1) -> /power stage/MOS_TEMP
- R64 pad 1: GND -> GNDA
- R84 pad 1: Net-(C116-Pad1) -> Net-(J15-Pad1)
- R84 pad 2: Net-(C117-Pad1) -> VDC
- R85 pad 1: Net-(IC1-Pad9) -> Net-(J15-Pad2)
- R85 pad 2: GND -> /io/IGNITION
- TH1 pad 1: Net-(FB3-Pad1) -> +3V3
- U1 pad 12: Net-(U1-Pad12) -> (no net)
- U1 pad 13: Net-(U1-Pad13) -> (no net)
- U1 pad 7: Net-(U1-Pad7) -> (no net)
- U11 pad 1: Net-(C93-Pad1) -> Net-(C100-Pad1)
- U12 pad 4: Net-(U12-Pad4) -> (no net)
- U2 pad 12: Net-(U3-Pad12) -> (no net)
- U2 pad 13: Net-(U3-Pad13) -> (no net)
- U2 pad 7: Net-(U3-Pad7) -> (no net)
- U3 pad 12: Net-(U5-Pad12) -> (no net)
- U3 pad 13: Net-(U5-Pad13) -> (no net)
- U3 pad 7: Net-(U5-Pad7) -> (no net)
- U4 pad 6: Net-(C28-Pad1) -> /power stage/VSUPA_U
- U4 pad 7: +3V3 -> /power stage/VSUPA_U
- U5 pad 6: Net-(C46-Pad1) -> /power stage/VSUPA_V
- U5 pad 7: +3V3 -> /power stage/VSUPA_V
- U6 pad 2: Net-(U6-Pad2) -> GNDA
- U6 pad 3: Net-(U6-Pad2) -> GNDA
- U6 pad 4: Net-(U6-Pad2) -> GNDA
- U6 pad 6: Net-(C59-Pad1) -> /power stage/VSUPA_W
- U6 pad 7: +3V3 -> /power stage/VSUPA_W
- U8 pad 2: Net-(U7-Pad2) -> (no net)
- U8 pad 25: /mcu/ADC15 -> (no net)
- U8 pad 28: Net-(U7-Pad28) -> (no net)
- U8 pad 3: Net-(U7-Pad3) -> (no net)
- U8 pad 33: Net-(U7-Pad33) -> (no net)
- U8 pad 4: Net-(U7-Pad4) -> (no net)
- U8 pad 40: Net-(U7-Pad40) -> (no net)
- U8 pad 50: Net-(U7-Pad50) -> (no net)
- U8 pad 51: Net-(U7-Pad51) -> (no net)
- U8 pad 52: Net-(U7-Pad52) -> (no net)
- U8 pad 53: Net-(U7-Pad53) -> (no net)
- U8 pad 54: Net-(U7-Pad54) -> (no net)
- U8 pad 55: Net-(U7-Pad55) -> (no net)
- U8 pad 56: Net-(U7-Pad56) -> (no net)
- U8 pad 59: /mcu/FAULT -> (no net)
Routing:
- net +12V: track 4.98 -> 108.8 mm, vias 0 -> 40
- net GND: track 4.87 -> 82.5 mm, vias 112 -> 217
- net +3V3: track 0.00 -> 74.5 mm, vias 0 -> 12
- net /pwr mng/SW: track 0.00 -> 62.0 mm, vias 0 -> 26
- net Net-(R29-Pad1): track 0.00 -> 54.3 mm, vias 0 -> 1
- net Net-(R30-Pad1): track 0.00 -> 54.2 mm, vias 0 -> 1
- net Net-(R27-Pad1): track 64.4 -> 111.6 mm, vias 1 -> 4
- net /power stage/MOS_TEMP: track 0.00 -> 33.7 mm, vias 0 -> 1
- net Net-(R26-Pad1): track 76.7 -> 110.3 mm, vias 1 -> 4
- net VDC: track 0.00 -> 28.7 mm, vias 117 -> 140
- net /mcu/ISENSE_U: track 0.00 -> 25.6 mm
- net /io/IGNITION: track 0.00 -> 22.0 mm, vias 0 -> 2
- net GNDA: track 0.00 -> 20.6 mm, vias 0 -> 13
- net /pwr mng/BOTTOM_GATE: track 0.00 -> 19.9 mm, vias 0 -> 1
- net /pwr mng/INTVCC: track 0.00 -> 12.7 mm, vias 0 -> 2
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- added copper zone on In1.Cu, net (none)
- added copper zone on B.Cu, net +12V
- added copper zone on F.Cu, net +12V
- added copper zone on In1.Cu, net +12V
- added copper zone on B.Cu, net +3V3
- added copper zone on F.Cu, net +3V3
- added copper zone on In1.Cu, net +3V3
- added copper zone on F.Cu, net +5V
- added copper zone on B.Cu, net /power stage/PHASE_V
- added copper zone on B.Cu, net /power stage/PHASE_W
- added copper zone on B.Cu, net /power stage/VBOOT_U
- added copper zone on B.Cu, net /power stage/VBOOT_V
- added copper zone on B.Cu, net /power stage/VBOOT_W
- added copper zone on F.Cu, net /power stage/VSUPA_U
- added copper zone on F.Cu, net /power stage/VSUPA_V
- added copper zone on F.Cu, net /power stage/VSUPA_W
- added copper zone on B.Cu, net /pwr mng/SW
- added copper zone on F.Cu, net /pwr mng/SW
- added copper zone on In1.Cu, net /pwr mng/SW
- added copper zone on F.Cu, net GNDA
- added copper zone on In1.Cu, net GNDA
- added copper zone on B.Cu, net Net-(C100-Pad1)
Other:
- board size 231 x 75 mm -> 231 x 67 mm
- net class Default: clearance 0.2 -> 0.16
- rule trace_clearance: 0.2 -> 0.16

Commit message: finished routing
Parts:
- removed FB6: Ferrite_Bead_Small, Inductor_SMD:L_0603_1608Metric
- C62, C64, C68, C70, C72, C73, C74, C79, C80, R69, Y1: moved to B.Cu
- J16: value Conn_01x04 -> CAN
- U9: footprint Package_TO_SOT_SMD:SOT-23-6 -> Package_TO_SOT_SMD:SOT-666
- moved R73 78.7 mm to (86.0, -11.5)
- moved C84 73.6 mm to (86.0, -13.5), turned to 180 degrees
- moved R75 68.6 mm to (79.0, -13.5)
- moved C86 68.5 mm to (79.0, -11.5), turned to 180 degrees
- moved D4 68.0 mm to (176.5, -3.25)
- moved D5 68.0 mm to (179.5, -3.25)
- moved D6 68.0 mm to (182.5, -3.25)
- moved R70 68.0 mm to (176.5, -6.75)
- moved R71 68.0 mm to (179.5, -6.96)
- moved R72 68.0 mm to (182.5, -6.75)
- moved R80 63.4 mm to (82.5, -13.5)
- moved C87 58.0 mm to (82.5, -11.5), turned to 180 degrees
- moved C75 51.9 mm to (138.2, -16.2), turned to 90 degrees
- moved C69 51.6 mm to (136.8, -16.2), turned to 90 degrees
- moved FB7 50.6 mm to (150.2, -21.0), turned to 180 degrees
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Connections:
- C31 pad 2: GNDA -> GND
- C32 pad 2: GNDA -> GND
- C33 pad 2: GNDA -> GND
- C34 pad 2: GNDA -> GND
- C35 pad 2: GNDA -> GND
- C36 pad 2: GNDA -> GND
- C37 pad 2: GNDA -> GND
- C38 pad 2: GNDA -> GND
- C39 pad 2: GNDA -> GND
- C54 pad 2: GNDA -> GND
- C62 pad 1: Net-(C62-Pad1) -> +3V3
- C64 pad 1: Net-(C62-Pad1) -> +3V3
- C65 pad 1: GNDA -> GND
- C66 pad 1: GNDA -> GND
- C67 pad 1: GNDA -> GND
- C68 pad 1: Net-(C62-Pad1) -> +3V3
- C69 pad 1: Net-(C62-Pad1) -> +3V3
- C70 pad 1: Net-(C62-Pad1) -> +3V3
- C71 pad 1: Net-(C62-Pad1) -> +3V3
- C75 pad 1: Net-(C62-Pad1) -> +3V3
- C77 pad 1: Net-(C62-Pad1) -> +3V3
- C79 pad 1: Net-(C62-Pad1) -> +3V3
- C80 pad 1: Net-(C62-Pad1) -> +3V3
- C81 pad 2: GNDA -> GND
- C82 pad 2: GNDA -> GND
- C83 pad 2: GNDA -> GND
- C86 pad 2: GNDA -> GND
- C87 pad 2: GNDA -> GND
- H1 pad 1: GNDS -> Net-(H1-Pad1)
- H2 pad 1: GNDS -> Net-(H2-Pad1)
- H3 pad 1: GNDS -> Net-(H3-Pad1)
- H4 pad 1: GNDS -> Net-(H4-Pad1)
- H7 pad 1: GNDS -> GND
- H9 pad 1: GNDS -> Net-(H9-Pad1)
- J11 pad 3: GNDA -> GND
- J13 pad 3: GNDA -> GND
- R53 pad 1: GNDA -> GND
- R55 pad 1: GNDA -> GND
- R57 pad 1: GNDA -> GND
- R60 pad 1: GNDA -> GND
- R64 pad 1: GNDA -> GND
- U4 pad 2: GNDA -> GND
- U4 pad 3: GNDA -> GND
- U4 pad 4: GNDA -> GND
- U5 pad 2: GNDA -> GND
- U5 pad 3: GNDA -> GND
- U5 pad 4: GNDA -> GND
- U6 pad 2: GNDA -> GND
- U6 pad 3: GNDA -> GND
- U6 pad 4: GNDA -> GND
- U8 pad 1: Net-(C62-Pad1) -> +3V3
- U8 pad 12: GNDA -> GND
- U8 pad 19: Net-(C62-Pad1) -> +3V3
- U8 pad 32: Net-(C62-Pad1) -> +3V3
- U8 pad 48: Net-(C62-Pad1) -> +3V3
- U8 pad 64: Net-(C62-Pad1) -> +3V3
- U9 pad 1: Net-(J10-Pad2) -> Net-(R77-Pad1)
- U9 pad 4: Net-(R77-Pad1) -> Net-(J10-Pad2)
Routing:
- net +12V: track 108.8 -> 327.9 mm, vias 40 -> 41
- net /mcu/DISABLE: track 0.00 -> 156.3 mm, vias 0 -> 5
- net GND: track 82.5 -> 209.2 mm, vias 217 -> 241
- net /mcu/PWM_W_HIGH: track 0.00 -> 103.3 mm, vias 0 -> 2
- net /mcu/PWM_W_LOW: track 0.00 -> 101.7 mm, vias 0 -> 2
- net /mcu/USENSE_W: track 3.02 -> 103.8 mm, vias 0 -> 2
- net /mcu/ISENSE_U: track 25.6 -> 119.7 mm, vias 0 -> 4
- net /mcu/SCK_ADC_EXT: track 0.00 -> 79.8 mm, vias 0 -> 2
- net +5V: track 4.66 -> 76.0 mm
- net /mcu/MISO_ADC_EXT2: track 0.00 -> 70.5 mm, vias 0 -> 2
- net /io/RC_PWM: track 0.00 -> 67.2 mm, vias 0 -> 2
- net /io/RX: track 0.00 -> 61.5 mm, vias 0 -> 2
- net /io/MOTOR_TEMP: track 0.00 -> 59.3 mm, vias 0 -> 2
- net /io/TX: track 0.00 -> 58.4 mm, vias 0 -> 2
- net /mcu/USENSE_U: track 2.77 -> 58.8 mm, vias 0 -> 2
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- removed copper zone on In1.Cu, net (none)
- removed copper zone on F.Cu, net GNDA
- removed copper zone on In1.Cu, net GNDA
Other:
- net class Default: trace_width 0.25 -> 0.2
- net class high voltage added: clearance 0.3, trace_width 0.2, via_dia 0.8, via_drill 0.4
- board text added: "3V3"
- board text added: "ERR"
- board text added: "THR"
